Commit message: working camera, needs debugging

File: sensors/urdf/wamv_with_zed2.xacro (robot description, xacro)
@@ -1,19 +1,8 @@
 <?xml version="1.0"?>
-<sdf version="1.9">
-  <model name="wamv_with_zed2">
-    <include>
-      <!-- Bring in the base WAM-V from VRX -->
-      <uri>model://wamv</uri>
-    </include>
-    <include>
-      <!-- Bring in your ZED2 camera from your own package -->
-      <uri>model://zed2_camera</uri>
-      <pose>0.3 0 1.2 0 0 0</pose>
-    </include>
-    <!-- Fixed joint to attach ZED2 to WAM-V -->
-    <joint name="wamv_zed2_fixed_joint" type="fixed">
-      <parent>wamv::base_link</parent>
-      <child>zed2_camera::zed2_link</child>
-    </joint>
-  </model>
-</sdf>
+<!-- Thin wrapper: reuse canonical VRX WAM-V model and only add ZED2 -->
+<robot xmlns:xacro="http://ros.org/wiki/xacro" name="wamv_with_zed2">
+  <xacro:include filename="$(find wamv_gazebo)/urdf/wamv_gazebo.urdf.xacro"/>
+  <xacro:include filename="$(find galaxsea)/sensors/urdf/zed2_camera.xacro"/>
+  <!-- Attach ZED2 into the same namespaced model tree as the canonical WAM-V -->
+  <xacro:zed2_camera parent_link="$(arg namespace)/base_link" xyz="0.3 0 1.2" rpy="0 0 0" namespace="$(arg namespace)" />
+</robot>

File: sensors/urdf/zed2_camera.xacro (robot description, xacro)
@@ -1,32 +1,85 @@
 <?xml version="1.0"?>
-<robot xmlns:xacro="http://www.ros.org/wiki/xacro">
-  <!-- ZED2 Camera Macro -->
-  <xacro:macro name="zed2_camera" params="parent_link xyz:='0 0 0' rpy:='0 0 0'">
-    <!-- Visual -->
-    <link name="zed2_link">
+<robot xmlns:xacro="http://ros.org/wiki/xacro">
+  <xacro:macro name="zed2_camera" params="parent_link:='wamv/base_link' xyz:='0 0 0' rpy:='0 0 0' namespace:='wamv'">
+    <!-- ================================================================
+         ZED2 Left Camera Link (primary / reference frame)
+         Real ZED2 body: 175mm x 30mm x 33mm, 159g
+    ================================================================ -->
+    <link name="${namespace}/zed2_link">
       <visual>
+        <origin xyz="0 0 0" rpy="0 0 ${pi/2}"/>
         <geometry>
-          <!-- Replace this mesh with an actual one if available -->
-          <!-- <mesh filename="package://my_robot_sensors/meshes/zed2.dae" scale="1 1 1"/> -->
+          <box size="0.175 0.03 0.033"/>
         </geometry>
+        <material name="zed2_body">
+          <color rgba="0.1 0.1 0.1 1.0"/>
+        </material>
       </visual>
+      <collision>
+        <origin xyz="0 0 0" rpy="0 0 0"/>
+        <geometry>
+          <box size="0.175 0.03 0.033"/>
+        </geometry>
+      </collision>
       <inertial>
-        <mass value="0.2"/>
+        <mass value="0.159"/>
         <origin xyz="0 0 0" rpy="0 0 0"/>
-        <inertia ixx="0.0001" iyy="0.0001" izz="0.0001" ixy="0" ixz="0" iyz="0"/>
+        <!-- Inertia for a solid box: m/12*(b²+c²), etc. -->
+        <inertia
+          ixx="0.000033" iyy="0.000041" izz="0.000065"
+          ixy="0" ixz="0" iyz="0"/>
       </inertial>
     </link>
-    <!-- Fixed Joint -->
-    <joint name="zed2_joint" type="fixed">
+    <joint name="${namespace}/zed2_joint" type="fixed">
       <parent link="${parent_link}"/>
-      <child link="zed2_link"/>
+      <child link="${namespace}/zed2_link"/>
       <origin xyz="${xyz}" rpy="${rpy}"/>
     </joint>
-    <!-- Gazebo sensor plugin -->
-    <gazebo reference="zed2_link">
-      <sensor name="zed2_depth_camera" type="depth_camera">
+    <!-- ================================================================
+         ZED2 Right Camera Link  (120mm stereo baseline offset)
+    ================================================================ -->
+    <link name="${namespace}/zed2_right_link">
+      <inertial>
+        <mass value="0.001"/>
+        <origin xyz="0 0 0" rpy="0 0 0"/>
+        <inertia ixx="0.000001" iyy="0.000001" izz="0.000001"
+                 ixy="0" ixz="0" iyz="0"/>
+      </inertial>
+    </link>
+    <joint name="${namespace}/zed2_right_joint" type="fixed">
+      <parent link="${namespace}/zed2_link"/>
+      <child link="${namespace}/zed2_right_link"/>
+      <!-- ZED2 baseline: 120mm in -Y (camera convention) -->
+      <origin xyz="0 -0.12 0" rpy="0 0 0"/>
+    </joint>
+    <!-- ================================================================
+         Optical frame links (Z forward, X right, Y down — ROS convention)
+    ================================================================ -->
+    <link name="${namespace}/zed2_left_optical_frame"/>
+    <joint name="${namespace}/zed2_left_optical_joint" type="fixed">
+      <parent link="${namespace}/zed2_link"/>
+      <child link="${namespace}/zed2_left_optical_frame"/>
+      <origin xyz="0 0 0" rpy="0 0 0"/>
+    </joint>
+    <link name="${namespace}/zed2_right_optical_frame"/>
+    <joint name="${namespace}/zed2_right_optical_joint" type="fixed">
+      <parent link="${namespace}/zed2_right_link"/>
+      <child link="${namespace}/zed2_right_optical_frame"/>
+      <origin xyz="0 0 0" rpy="0 0 0"/>
+    </joint>
+    <!-- ================================================================
+         Gazebo Sensors
+    ================================================================ -->
+    <gazebo reference="${namespace}/zed2_link">
+      <!-- ================================================================
+           LEFT RGB Camera  (30 Hz, 1280x720, with Gaussian noise)
+      ================================================================ -->
+      <sensor name="zed2_left_rgb" type="camera">
+        <always_on>true</always_on>
         <update_rate>30</update_rate>
-        <camera>
-          <horizontal_fov>1.3962634</horizontal_fov>
+        <visualize>false</visualize>
+        <topic>/zed2/left/image_rect_color</topic>
+        <camera>
+          <horizontal_fov>1.8325957</horizontal_fov>  <!-- ZED2: ~105° HFOV -->
           <image>
             <width>1280</width>
@@ -35,22 +88,166 @@
           </image>
           <clip>
-            <near>0.1</near>
-            <far>20.0</far>
-          </clip>
-        </camera>
-        <plugin name="zed2_camera_plugin" filename="libgazebo_ros_camera.so">
-          <ros>
-            <namespace>/zed2</namespace>
-          </ros>
-          <camera_name>zed2</camera_name>
-          <frame_name>zed2_link</frame_name>
-        </plugin>
-        <plugin name="zed2_depth_plugin" filename="libgazebo_ros_depth_camera.so">
-          <ros>
-            <namespace>/zed2</namespace>
-          </ros>
-          <camera_name>zed2_depth</camera_name>
-          <frame_name>zed2_link</frame_name>
-        </plugin>
+            <near>0.2</near>
+            <far>20.0</far>
+          </clip>
+          <noise>
+            <type>gaussian</type>
+            <mean>0.0</mean>
+            <stddev>0.007</stddev>
+          </noise>
+          <distortion>
+            <k1>0.0</k1>
+            <k2>0.0</k2>
+            <k3>0.0</k3>
+            <p1>0.0</p1>
+            <p2>0.0</p2>
+            <center>0.5 0.5</center>
+          </distortion>
+          <optical_frame_id>${namespace}/${namespace}/zed2_left_optical_frame</optical_frame_id>
+        </camera>
+      </sensor>
+      <!-- ================================================================
+           DEPTH Camera  — correct format: R_FLOAT32, 15 Hz
+           ZED2 depth range: 0.2 m – 20 m
+      ================================================================ -->
+      <sensor name="zed2_depth" type="depth_camera">
+        <always_on>true</always_on>
+        <update_rate>15</update_rate>
+        <visualize>false</visualize>
+        <topic>/zed2/depth/depth_registered</topic>
+        <camera>
+          <horizontal_fov>1.8325957</horizontal_fov>
+          <image>
+            <width>1280</width>
+            <height>720</height>
+            <format>R_FLOAT32</format>  <!-- FIXED: was R8G8B8, wrong for depth -->
+          </image>
+          <clip>
+            <near>0.2</near>
+            <far>20.0</far>
+          </clip>
+          <noise>
+            <type>gaussian</type>
+            <mean>0.0</mean>
+            <stddev>0.004</stddev>  <!-- ~4mm depth noise, realistic for ZED2 -->
+          </noise>
+          <optical_frame_id>${namespace}/${namespace}/zed2_left_optical_frame</optical_frame_id>
+        </camera>
+      </sensor>
+      <!-- ================================================================
+           RGBD / Point Cloud  (10 Hz — expensive, keep rate low)
+           Publishes sensor_msgs/PointCloud2 on GZ transport
+      ================================================================ -->
+      <sensor name="zed2_point_cloud" type="rgbd_camera">
+        <always_on>true</always_on>
+        <update_rate>10</update_rate>
+        <visualize>false</visualize>
+        <topic>/zed2/point_cloud/cloud_registered</topic>
+        <camera>
+          <horizontal_fov>1.8325957</horizontal_fov>
+          <image>
+            <width>1280</width>
+            <height>720</height>
+            <format>R8G8B8</format>
+          </image>
+          <clip>
+            <near>0.2</near>
+            <far>20.0</far>
+          </clip>
+          <optical_frame_id>${namespace}/${namespace}/zed2_left_optical_frame</optical_frame_id>
+        </camera>
+      </sensor>
+      <!-- ================================================================
+           IMU  (ZED2 built-in: ICM-42688-P equivalent, 400 Hz)
+           Placed at the IMU origin, coincident with the camera body.
+      ================================================================ -->
+      <sensor name="zed2_imu" type="imu">
+        <always_on>true</always_on>
+        <update_rate>400</update_rate>
+        <topic>/zed2/imu/data</topic>
+        <imu>
+          <angular_velocity>
+            <x>
+              <noise type="gaussian">
+                <mean>0.0</mean>
+                <stddev>0.005</stddev>    <!-- rad/s -->
+                <bias_mean>0.0001</bias_mean>
+                <bias_stddev>0.000075</bias_stddev>
+              </noise>
+            </x>
+            <y>
+              <noise type="gaussian">
+                <mean>0.0</mean>
+                <stddev>0.005</stddev>
+                <bias_mean>0.0001</bias_mean>
+                <bias_stddev>0.000075</bias_stddev>
+              </noise>
+            </y>
+            <z>
+              <noise type="gaussian">
+                <mean>0.0</mean>
+                <stddev>0.005</stddev>
+                <bias_mean>0.0001</bias_mean>
+                <bias_stddev>0.000075</bias_stddev>
+              </noise>
+            </z>
+          </angular_velocity>
+          <linear_acceleration>
+            <x>
+              <noise type="gaussian">
+                <mean>0.0</mean>
+                <stddev>0.02</stddev>    <!-- m/s² -->
+                <bias_mean>0.01</bias_mean>
+                <bias_stddev>0.001</bias_stddev>
+              </noise>
+            </x>
+            <y>
+              <noise type="gaussian">
+                <mean>0.0</mean>
+                <stddev>0.02</stddev>
+                <bias_mean>0.01</bias_mean>
+                <bias_stddev>0.001</bias_stddev>
+              </noise>
+            </y>
+            <z>
+              <noise type="gaussian">
+                <mean>0.0</mean>
+                <stddev>0.02</stddev>
+                <bias_mean>0.01</bias_mean>
+                <bias_stddev>0.001</bias_stddev>
+              </noise>
+            </z>
+          </linear_acceleration>
+        </imu>
+      </sensor>
+    </gazebo>
+    <!-- Right camera sensor lives on the right link -->
+    <gazebo reference="${namespace}/zed2_right_link">
+      <!-- ================================================================
+           RIGHT RGB Camera  (30 Hz — stereo pair with left)
+      ================================================================ -->
+      <sensor name="zed2_right_rgb" type="camera">
+        <always_on>true</always_on>
+        <update_rate>30</update_rate>
+        <visualize>false</visualize>
+        <topic>/zed2/right/image_rect_color</topic>
+        <camera>
+          <horizontal_fov>1.8325957</horizontal_fov>
+          <image>
+            <width>1280</width>
+            <height>720</height>
+            <format>R8G8B8</format>
+          </image>
+          <clip>
+            <near>0.2</near>
+            <far>20.0</far>
+          </clip>
+          <noise>
+            <type>gaussian</type>
+            <mean>0.0</mean>
+            <stddev>0.007</stddev>
+          </noise>
+          <optical_frame_id>${namespace}/${namespace}/zed2_right_optical_frame</optical_frame_id>
+        </camera>
       </sensor>
     </gazebo>
